File: Electronics/IMUnav_Gravi_Addon/IMUnav_Gravi_Addon.kicad_sch (KiCad schematic)
At the start: 5 parts, among them J1 Conn_01x03_Pin, J2 Conn_01x03_Pin, J3 Conn_02x08_Odd_Even, J4 Conn_01x03_Socket, U1 MT3608-module

Commit message: addon pcb routing
Parts:
- added H1, H2: MountingHole, MountingHole:MountingHole_3.2mm_M3, symbol Mechanical:MountingHole
- added J5: BMP280-module, Connector_PinSocket_2.54mm:PinSocket_1x06_P2.54mm_Vertical, symbol Connector:Conn_01x06_Pin
- added JP1, JP2: SolderJumper_3_Bridged12, Jumper:SolderJumper-3_P1.3mm_Bridged12_RoundedPad1.0x1.5mm_NumberLabels, symbol Jumper:SolderJumper_3_Bridged12
Connections:
- net +3V3: now also J5.1 (Pin_1), JP1.3 (B), JP2.1 (A)
- net GND: now also J5.2 (Pin_2), JP1.1 (A), JP2.3 (B)
- net SCL: now also J5.3 (Pin_3)
- net SDA: now also J5.4 (Pin_4)
- new net CSB: J5.5 (Pin_5), JP2.2 (C)
- new net SDO: J5.6 (Pin_6), JP1.2 (C)
